File: hardware/electronics/pcb/v4/solenoid_driver.kicad_pcb (KiCad board)
At the start: 2 copper layers, 78 x 87 mm, 29 parts, among them Q1 IRLZ44N, Q2 IRLZ44N, Q3 IRLZ44N, Q4 IRLZ44N

Commit message: feat: created v4 pcb
Parts:
- moved R6 15.0 mm to (105.0, 95.0), turned to 0 degrees
- moved R4 14.7 mm to (104.9, 80.0), turned to 0 degrees
- moved R2 14.4 mm to (104.9, 65.5), turned to 0 degrees
- moved R8 14.4 mm to (104.9, 110.5), turned to 0 degrees
- moved Q2 7.61 mm to (96.5, 85.0)
- moved R7 7.54 mm to (115.1, 115.5), turned to 180 degrees
- moved Q1 7.52 mm to (96.5, 70.5)
- moved R1 7.51 mm to (115.0, 70.5), turned to 180 degrees
- moved Q3 7.17 mm to (96.5, 100.0)
- moved R3 7.07 mm to (115.1, 85.0), turned to 180 degrees
- moved Q4 7.06 mm to (96.5, 115.5)
- moved R5 6.60 mm to (115.1, 100.0), turned to 180 degrees
Connections:
- R8 pad 1: GND -> Net-(Q4-G)
Routing:
- net Net-(Q4-G): track 21.6 -> 13.5 mm
- net Net-(Q1-G): track 21.6 -> 13.5 mm
- net Net-(Q2-G): track 21.6 -> 13.6 mm
- net Net-(Q3-G): track 21.6 -> 13.6 mm
- net Net-(D2-A): track 37.1 -> 29.1 mm
- net Net-(D1-A): track 36.7 -> 29.0 mm
- net Net-(D3-A): track 35.9 -> 28.3 mm
- net Net-(D4-A): track 32.9 -> 25.7 mm
- net /SOL4: track 22.2 -> 28.2 mm
- net /SOL1: track 20.7 -> 15.3 mm
- net /SOL2: track 16.6 -> 13.6 mm
- net +12V: track 182.9 -> 182.1 mm
- added copper zone on B.Cu, net GND
- removed copper zone on F.Cu, net GND
Other:
- board size 78 x 87 mm -> 78 x 82.5 mm
- board text removed: "1.5"

Commit message: docs: enhanced hardware READMEs
Parts:
- R9: value 1k -> 2k
Changed lines of the file:
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@@
 			)
 		)
-		(property "Value" "1k"
+		(property "Value" "2k"
 			(at 5.08 2.37 0)
 			(layer "F.Fab")
