File: hardware/electronics/pcb/v4/solenoid_driver.kicad_sch (KiCad schematic)
At the start: 25 parts, among them Q1 IRLZ44N, Q2 IRLZ44N, Q3 IRLZ44N, Q4 IRLZ44N

Commit message: docs: enhanced hardware READMEs
Parts:
- R9: value 1k -> 2k
Changed lines of the file:
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@@
 			)
 		)
-		(property "Value" "1k"
+		(property "Value" "2k"
 			(at 147.32 46.736 90)
 			(show_name no)
